Commit message: updated urdf with laser and camera

File: create_description/urdf/create_2.urdf.xacro (robot description, xacro)
@@ -3,6 +3,43 @@
   <xacro:include filename="$(find create_description)/urdf/create_base.urdf.xacro" />
   <xacro:include filename="$(find create_description)/urdf/create_2_gazebo.urdf.xacro" />
+    <xacro:property name="M_SCALE" value="0.001"/>
   <xacro:create_base wheel_separation="0.235" base_diameter="0.3485">
-    <mesh filename="package://create_description/meshes/create_2.dae" />
+    <mesh filename="package://create_description/meshes/shoebot_collision.stl" scale="${M_SCALE} ${M_SCALE} ${M_SCALE}"/>
   </xacro:create_base>
+    <link name="laser">
+        <inertial>
+            <mass value="0.00833634573995571"/>
+            <inertia ixx="1.01866461240801E-06" ixy="-5.88447626567756E-08" ixz="7.83857244757914E-08"
+                     iyy="5.10039589974707E-07" iyz="-7.12664289617235E-09" izz="1.28270671527309E-06"/>
+        </inertial>
+    </link>
+    <joint name="base_to_laser" type="fixed">
+        <parent link="base_link"/>
+        <child link="laser"/>
+        <origin xyz="-0.091987 0 0.5" rpy="0 0 0"/>
+    </joint>
+    <link name="camera1">
+        <inertial>
+            <mass value="0.00833634573995571"/>
+            <inertia ixx="1.01866461240801E-06" ixy="-5.88447626567756E-08" ixz="7.83857244757914E-08"
+                     iyy="5.10039589974707E-07" iyz="-7.12664289617235E-09" izz="1.28270671527309E-06"/>
+        </inertial>
+    </link>
+    <joint name="base_to_camera1" type="fixed">
+        <parent link="base_link"/>
+        <child link="camera1"/>
+        <origin xyz="-0.041986 0 0.454529" rpy="0 0 0"/>
+    </joint>
+    <link name="camera2">
+        <inertial>
+            <mass value="0.00833634573995571"/>
+            <inertia ixx="1.01866461240801E-06" ixy="-5.88447626567756E-08" ixz="7.83857244757914E-08"
+                     iyy="5.10039589974707E-07" iyz="-7.12664289617235E-09" izz="1.28270671527309E-06"/>
+        </inertial>
+    </link>
+    <joint name="base_to_camera2" type="fixed">
+        <parent link="base_link"/>
+        <child link="camera2"/>
+        <origin xyz="-0.053586 0 0.43102" rpy="0 0.523599 0"/>
+    </joint>
 </robot>

File: create_description/urdf/create_base.urdf.xacro (robot description, xacro)
@@ -53,5 +53,5 @@
     </inertial>
     <visual>
-      <origin xyz=" 0 0 0.0308" rpy="0 0 0" />
+      <origin xyz=" 0 0 0" rpy="1.57 0 1.57" />
       <geometry>
         <xacro:insert_block name="mesh" />

Commit message: getting new urdf working with nav

File: create_description/urdf/create_2.urdf.xacro (robot description, xacro)
@@ -7,5 +7,5 @@
     <mesh filename="package://create_description/meshes/shoebot_collision.stl" scale="${M_SCALE} ${M_SCALE} ${M_SCALE}"/>
   </xacro:create_base>
-    <link name="laser">
+    <link name="laser_link">
         <inertial>
             <mass value="0.00833634573995571"/>
@@ -16,8 +16,8 @@
     <joint name="base_to_laser" type="fixed">
         <parent link="base_link"/>
-        <child link="laser"/>
+        <child link="laser_link"/>
         <origin xyz="-0.091987 0 0.5" rpy="0 0 0"/>
     </joint>
-    <link name="camera1">
+    <link name="camera1_link">
         <inertial>
             <mass value="0.00833634573995571"/>
@@ -28,8 +28,8 @@
     <joint name="base_to_camera1" type="fixed">
         <parent link="base_link"/>
-        <child link="camera1"/>
+        <child link="camera1_link"/>
         <origin xyz="-0.041986 0 0.454529" rpy="0 0 0"/>
     </joint>
-    <link name="camera2">
+    <link name="camera2_link">
         <inertial>
             <mass value="0.00833634573995571"/>
@@ -40,5 +40,5 @@
     <joint name="base_to_camera2" type="fixed">
         <parent link="base_link"/>
-        <child link="camera2"/>
+        <child link="camera2_link"/>
         <origin xyz="-0.053586 0 0.43102" rpy="0 0.523599 0"/>
     </joint>
